File: daqduino.kicad_sch (KiCad schematic)
At the start: 4 parts

Commit message: khnljkglkuv
Parts:
- removed PT1: 5k, Potentiometer_THT:Potentiometer_Alpha_RD901F-40-00D_Single_Vertical_CircularHoles, symbol 000_Resistors_Immo:Alpha Pot
- added PT1: 5kB, 000 Resistors Immo:16MM_CENTERMOUNT, symbol 000_Resistors_Immo:16mm Pot
- added TP1, TP2: TestPoint, symbol Connector:TestPoint
- R3: value 100M -> 1M
Connections:
- net +24V: now also TP1.1
- net CURRENT_SENSE_A: now also PT1.3, TP2.1
- net at R1.2: now also PT1.1, PT1.2
Other:
- note added: "-14.3 uA"
- note added: "20.38 mA"
- note added: "20.39 mA"
- note added: "23.88 V"
- note added: "31.2 mV"
- moved on the sheet: R1, R2, R3
