File: daqduino-pcb/daqduino.kicad_sch (KiCad schematic)
At the start: 6 parts

Commit message: ksdflk
Parts:
- removed PT1: 5kB, 000 Resistors Immo:16MM_CENTERMOUNT, symbol 000_Resistors_Immo:16mm Pot
- removed R1: 1k2, Resistor_SMD:R_0805_2012Metric_Pad1.20x1.40mm_HandSolder, symbol 000_Resistors_Immo:Resistor_0805
- removed R2: 1r, Resistor_SMD:R_0805_2012Metric_Pad1.20x1.40mm_HandSolder, symbol 000_Resistors_Immo:Resistor_0805
- removed R3: 1M, Resistor_SMD:R_0805_2012Metric_Pad1.20x1.40mm_HandSolder, symbol 000_Resistors_Immo:Resistor_0805
- removed TP1, TP2: TestPoint, symbol Connector:TestPoint
- added C1: 470n, symbol Device:C
- added R1: 250r, symbol Device:R
- added U1 (x2): LM358, Package_SO:SOIC-8_3.9x4.9mm_P1.27mm, symbol Amplifier_Operational:LM358
Connections:
- new net +12V: U1.8 (V+)
- new net -12V: U1.4 (V-)
- new net CURRENT_SOURCE: C1.1, R1.1, U1.2 (-)
- new net GND: U1.3 (+)
- new net VOLTAGE_OUTPUT: C1.2, R1.2, U1.1
- no-connect marks 0 -> 1
Other:
- note added: "Desired Functions: - 10v, 12v and 24v outputs for sensor power - 0 - 10v analog input - 0 - 5v TTL IO - 4 - 20mA input - OLED Screen - Encoder Control - Basic Scaling Stretch Goals: - 0 - 10 v output - 0 - 20 mA output Communications: - Serial Data - Labveiw Integration? - Python App"
- note added: "TransImpedance Amplifer Circuit Sources: https://www.ti.com/lit/an/sboa268a/sboa268a.pdf?ts=1685014387183&ref_url=https%253A%252F%252Fwww.google.com%252F https://circuitdigest.com/tutorial/transimpedance-amplifier-design-working-and-applications"
- note removed: "-14.3 uA"
- note removed: "20.38 mA"
- note removed: "20.39 mA"
- note removed: "23.88 V"
- note removed: "31.2 mV"
- note removed: "Dummy Load"
- note removed: "Functions: - 10v, 12v and 24v outputs for sensor power - 0 - 10v analog input - 0 - 5v TTL IO - 4 - 20mA input - OLED Screen - Encoder Control - Basic Scaling Stretch Goals: - 0 - 10 v output - 0 - 20 mA output Communications: - Serial Data - Labveiw Integration?"
- note removed: "Shunt Resistor"

Commit message: update
Parts:
- removed U1: LM358, Package_SO:SOIC-8_3.9x4.9mm_P1.27mm, symbol Amplifier_Operational:LM358
- added EC1, EC2: 100u, Capacitor_SMD:CP_Elec_10x10, symbol 000_Capacitor_Electrolytic_Immo:100u
- added J1: 24v Power Input, TerminalBlock:TerminalBlock_Altech_AK300-2_P5.00mm, symbol 000_Connectors_Immo:Screw_Terminal_01x02
- added U2: L7812, Package_TO_SOT_THT:TO-220-3_Vertical, symbol Regulator_Linear:L7812
- added XA1: Arduino_Uno_R3_Shield, PCM_arduino-library:Arduino_Uno_R3_Shield, symbol PCM_arduino-library:Arduino_Uno_R3_Shield
- R1: value 250r -> 220r
Connections:
- net GND: now also EC1.2, EC2.2, J1.1 (Pin_1), U2.2 (GND); no longer U1.3 (+)
- new net 12V_BUS: EC2.1, U2.3 (OUT), XA1.VIN
- new net 24V_BUS: EC1.1, J1.2 (Pin_2), U2.1 (IN)
- new net 5V_BUS: XA1.5V1 (5V)
- new net BIAS_VOLTAGE: U1.3 (+)
- no-connect marks 1 -> 0
Other:
- note added: "#NOTE: 100r for + and - Current sensing, with virtual ground @ 2.5v"
- note added: "Desired Functions: - 10v, 12v and 24v outputs for sensor power - 0 - 10v analog input - 0 - 5v TTL IO - 4 - 20mA input Stretch Goals: - 0 - 10 v output - 0 - 20 mA output - OLED Screen - Encoder Control - Basic Scaling Communications: - Serial Data - Labveiw Integration? - Python App"
- note removed: "Desired Functions: - 10v, 12v and 24v outputs for sensor power - 0 - 10v analog input - 0 - 5v TTL IO - 4 - 20mA input - OLED Screen - Encoder Control - Basic Scaling Stretch Goals: - 0 - 10 v output - 0 - 20 mA output Communications: - Serial Data - Labveiw Integration? - Python App"
- moved on the sheet: U1B, U1C

Commit message: kjglkjhgkjhgf
Parts:
- added J2: Conn_2Rows-07Pins, symbol Connector_Generic:Conn_2Rows-07Pins
- added J3: Conn_02x06_Counter_Clockwise, symbol Connector_Generic:Conn_02x06_Counter_Clockwise
- added R2, R3: 10k, Resistor_SMD:R_0805_2012Metric_Pad1.20x1.40mm_HandSolder, symbol 000_Resistors_Immo:10k
Connections:
- net 5V_BUS: now also R2.2
- net GND: now also R3.1
- net V_ctrl: now reaches XA1.D5
- net at U1.5 (+): now also R2.1, R3.2
- net at U1.6 (-): now also U1.7, J3.1 (Pin_1)
Other:
- note added: "Bias Voltage Selection"
- moved on the sheet: U1B

Commit message: almost finished schematic
Parts:
- removed J2: Conn_2Rows-07Pins, symbol Connector_Generic:Conn_2Rows-07Pins
- removed J3: Conn_02x06_Counter_Clockwise, symbol Connector_Generic:Conn_02x06_Counter_Clockwise
- added C2: 100n, 000_Capacitors_Immo:C_0805_2012_HandSolder_kawaii, symbol 000_Capacitor_Film_Immo:100n
- added J2: Sense Current TestPoint, 000 Connectors Immo:TerminalBlock_Altech_AK300-2_P5.00mm, symbol 000_Connectors_Immo:Screw_Terminal_01x02
- added J3: Bias Voltage & Resistor Selection, symbol Connector_Generic:Conn_02x03_Counter_Clockwise
- added J4: Sensor Voltage Selection, symbol Connector_Generic:Conn_02x03_Counter_Clockwise
- added J5: 2 Wire Sensor (4-20mA), 000 Connectors Immo:TerminalBlock_Altech_AK300-2_P5.00mm, symbol 000_Connectors_Immo:Screw_Terminal_01x02
- added R4: 100r, symbol Device:R
- added TP1: Bias TestPoint, TestPoint:TestPoint_Bridge_Pitch2.54mm_Drill1.0mm, symbol Connector:TestPoint_Probe
- added TP2: 12v TestPoint, TestPoint:TestPoint_Bridge_Pitch2.54mm_Drill1.0mm, symbol Connector:TestPoint_Probe
- added TP3: 24v TestPoint, TestPoint:TestPoint_Bridge_Pitch2.54mm_Drill1.0mm, symbol Connector:TestPoint_Probe
- added TP4: 5v TestPoint, TestPoint:TestPoint_Bridge_Pitch2.54mm_Drill1.0mm, symbol Connector:TestPoint_Probe
- added TP5: Sense Voltage TestPoint, TestPoint:TestPoint_Bridge_Pitch2.54mm_Drill1.0mm, symbol Connector:TestPoint_Probe
- J1: PIN1 PIN1 -> gnd; PIN2 PIN2 -> 24v in
Connections:
- net +12V is gone; now on net 5V_BUS: U1.8 (V+)
- net -12V is gone; now on net GND: U1.4 (V-)
- net 12V_BUS: now also J4.5 (Pin_5), TP2.1
- net 24V_BUS: now also J4.1 (Pin_1), TP3.1
- net 5V_BUS: now also C2.1, J4.3 (Pin_3), TP4.1
- net BIAS_VOLTAGE: now also J3.2 (Pin_2)
- net GND: now also XA1.GND1 (GND), XA1.GND2 (GND), XA1.GND3 (GND), C2.2, J3.1 (Pin_1)
- net at U1.6 (-), U1.7: now also J3.3 (Pin_3), TP1.1
- net R_SET_B: now reaches XA1.A2
- net R_SET_B: now also C1.2, U1.1, J3.5 (Pin_5), TP5.1
- net CURRENT_SOURCE renamed R_SET_A
- net R_SET_A: now also R1.2, J2.2 (Pin_2), R4.2; no longer R1.1
- removed net VOLTAGE_OUTPUT: C1.2, R1.2, U1.1
- net V_ctrl renamed V_{ctrl}
- new net: J4.2 (Pin_2), J5.2 (Pin_2)
- new net: J3.4 (Pin_4), R4.1
- new net: J3.6 (Pin_6), R1.1
- new net SENSE_CURRENT: J2.1 (Pin_1), J5.1 (Pin_1)
- no-connect marks 0 -> 2
Other:
- note added: "#NOTE - Prototyping Feature Sense Current Terminal should be shorted with solid core wire during normal use. Open for testing sensor current input"
- note added: "#NOTE Feedforward resistor is set by Bias Voltage Selection Jumpers"
- note added: "1"
- note added: "2"
- note added: "3"
- note added: "4"
- note added: "5"
- note added: "6"
- note added: "Arduino Shield"
- note added: "Mode A"
- note added: "Mode B"
- note added: "Power Supply"
- note added: "Sensor Connection"
- note added: "Transimpediance Amplifyer"
- note added: "Use jumpers to select operational mode Mode A: Use for positive values of I_{in} for full resolution - 1 & 2 Bridged - 220r in circuit - 6 & 5 Bridged - Bias Set to GND Mode B: Use for positive or negative values of I_{in} with reduced resolution - 3 & 2 Bridged - 100r in circuit - 4 & 5 Bridged - Bias set to 1/2*V_{cc}"
- note added: "User Setting:"
- note added: "Voltage Selection"
- note removed: "#NOTE: 100r for + and - Current sensing, with virtual ground @ 2.5v"
- note removed: "TransImpedance Amplifer Circuit Sources: https://www.ti.com/lit/an/sboa268a/sboa268a.pdf?ts=1685014387183&ref_url=https%253A%252F%252Fwww.google.com%252F https://circuitdigest.com/tutorial/transimpedance-amplifier-design-working-and-applications"
- moved on the sheet: C1, EC1, EC2, J1, R2, R3, U1A, U1B, U1C, U2, XA1

Commit message: sdfsdf
Parts:
- added C3, C4: 100n, 000_Capacitors_Immo:C_0805_2012_HandSolder_kawaii, symbol 000_Capacitor_Film_Immo:100n
- added J6: Micro_SD_Card, Connector_Card:microSD_HC_Wuerth_693072010801, symbol Connector:Micro_SD_Card
- added R5, R6, R7, R8: 3k3, Resistor_SMD:R_0805_2012Metric_Pad1.20x1.40mm_HandSolder, symbol 000_Resistors_Immo:Resistor_0805
- added TP6: 3v3 TestPoint, TestPoint:TestPoint_Bridge_Pitch2.54mm_Drill1.0mm, symbol Connector:TestPoint_Probe
- added U3: TXS0108EPW, Package_SO:TSSOP-20_4.4x6.5mm_P0.65mm, symbol Logic_LevelTranslator:TXS0108EPW
Connections:
- net 5V_BUS: now also C3.1, U3.19 (VCCB)
- net GND: now also C3.2, C4.2, J6.6 (VSS), U3.11 (GND)
- net SENSOR_POWER: now reaches J4.2 (Pin_2), J5.2 (Pin_2)
- net 3V3_BUS: now reaches XA1.3V3 (3.3V)
- net 3V3_BUS: now also C4.1, J6.4 (VDD), R6.2, U3.2 (VCCA)
- net CHIP_SELECT: now reaches XA1.D10 (D10_CS)
- net CHIP_SELECT: now also R7.1
- net MOSI: now reaches XA1.D12
- net MOSI: now also R5.1
- net SCK: now reaches XA1.D13
- net SCK: now also R8.1
- net V_{ctrl}: no longer names the net of XA1.D5
- new net: R6.1, U3.10 (OE)
- new net: R8.2, U3.17 (B3)
- new net: R7.2, U3.18 (B2)
- new net: R5.2, U3.20 (B1)
- new net CLK: J6.5 (CLK), U3.4 (A3)
- new net CS: J6.2 (DAT3/CD), U3.3 (A2)
- new net D_{IN}: J6.3 (CMD), U3.1 (A1)
- no-connect marks 2 -> 4
Other:
- note added: "OE pulled to V_{ccA}"
- note added: "Sensor Voltage Selection Jumper For 24v Sensor: - Jumper pins 1 & 2 For 12v Sensor - Jumper pins 5 & 2 For 5v Sensor - Jumper pins 3 & 2 pins 4 & 6 NC"
- note added: "Use jumpers to select operational mode Mode A: Use for positive values of I_{in} for full resolution. - 1 & 2 Bridged - 220r in circuit - 6 & 5 Bridged - Bias Set to GND Mode B: Use for positive or negative values of I_{in} with reduced resolution. - 3 & 2 Bridged - 100r in circuit - 4 & 5 Bridged - Bias set to 1/2*V_{cc}"
- note added: "V_{ccA} <= V_{ccB}"
- note removed: "Use jumpers to select operational mode Mode A: Use for positive values of I_{in} for full resolution - 1 & 2 Bridged - 220r in circuit - 6 & 5 Bridged - Bias Set to GND Mode B: Use for positive or negative values of I_{in} with reduced resolution - 3 & 2 Bridged - 100r in circuit - 4 & 5 Bridged - Bias set to 1/2*V_{cc}"
- moved on the sheet: C1, C2, EC1, EC2, J1, J2, J3, J4, J5, R1, R2, R3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

Commit message: started pcb laypouty
Parts:
- removed C1: 470n, symbol Device:C
- removed J3: Bias Voltage & Resistor Selection, symbol Connector_Generic:Conn_02x03_Counter_Clockwise
- removed J4: Sensor Voltage Selection, symbol Connector_Generic:Conn_02x03_Counter_Clockwise
- removed J6: Micro_SD_Card, Connector_Card:microSD_HC_Wuerth_693072010801, symbol Connector:Micro_SD_Card
- removed R1: 220r, symbol Device:R
- removed R4: 100r, symbol Device:R
- removed TP6: 3v3 TestPoint, TestPoint:TestPoint_Bridge_Pitch2.54mm_Drill1.0mm, symbol Connector:TestPoint_Probe
- added C1: 470r, Capacitor_SMD:C_0805_2012Metric_Pad1.18x1.45mm_HandSolder, symbol 000_Capacitor_Film_Immo:cap_film_0805
- added D1: red, Diode_SMD:D_0805_2012Metric_Pad1.15x1.40mm_HandSolder, symbol 000_Diodes_Immo:LED_0805_smd
- added D2: yellow, Diode_SMD:D_0805_2012Metric_Pad1.15x1.40mm_HandSolder, symbol 000_Diodes_Immo:LED_0805_smd
- added D3: green, Diode_SMD:D_0805_2012Metric_Pad1.15x1.40mm_HandSolder, symbol 000_Diodes_Immo:LED_0805_smd
- added D4: blue, Diode_SMD:D_0805_2012Metric_Pad1.15x1.40mm_HandSolder, symbol 000_Diodes_Immo:LED_0805_smd
- added J3: Bias Voltage & Resistor Selection, 000_Pin_Headers_Immo:PinHeader_2x03_P2.54mm-alt-pin-no, symbol 000_Pin_Headers_Immo:Conn_02x03_Counter_Clockwise
- added J4: Sensor Voltage Selection, 000_Pin_Headers_Immo:PinHeader_2x03_P2.54mm-alt-pin-no, symbol 000_Pin_Headers_Immo:Conn_02x03_Counter_Clockwise
- added J7: Micro_SD_Card-molex, 000_Connectors_Immo:microSD_HC_Molex_104031-0811, symbol 000_Connectors_Immo:Micro_SD_Card-molex
- added R1: 220r, Resistor_SMD:R_0805_2012Metric_Pad1.20x1.40mm_HandSolder, symbol 000_Resistors_Immo:Resistor_0805
- added R10: 10k, Resistor_SMD:R_0805_2012Metric_Pad1.20x1.40mm_HandSolder, symbol 000_Resistors_Immo:10k
- added R11: 4k7, Resistor_SMD:R_0805_2012Metric_Pad1.20x1.40mm_HandSolder, symbol 000_Resistors_Immo:10k
- added R12: 2k2, Resistor_SMD:R_0805_2012Metric_Pad1.20x1.40mm_HandSolder, symbol 000_Resistors_Immo:10k
- added R13: 1k, Resistor_SMD:R_0805_2012Metric_Pad1.20x1.40mm_HandSolder, symbol 000_Resistors_Immo:10k
- added R4: 100r, Resistor_SMD:R_0805_2012Metric_Pad1.20x1.40mm_HandSolder, symbol 000_Resistors_Immo:100r
- added R9: 3k3, Resistor_SMD:R_0805_2012Metric_Pad1.20x1.40mm_HandSolder, symbol 000_Resistors_Immo:Resistor_0805
- added TP1: 24v TestPoint, TestPoint:TestPoint_Bridge_Pitch2.54mm_Drill1.0mm, symbol Connector:TestPoint_Probe
- J1: footprint TerminalBlock:TerminalBlock_Altech_AK300-2_P5.00mm -> 000_Connectors_Immo:TerminalBlock_Altech_AK300-2_P5.00mm; PIN2 24v in -> +24v
- J2: footprint 000 Connectors Immo:TerminalBlock_Altech_AK300-2_P5.00mm -> 000_Connectors_Immo:TerminalBlock_Altech_AK300-2_P5.00mm
- J5: footprint 000 Connectors Immo:TerminalBlock_Altech_AK300-2_P5.00mm -> 000_Connectors_Immo:TerminalBlock_Altech_AK300-2_P5.00mm; PIN1 - -> sense -; PIN2 + -> sense +
- TP3: value 24v TestPoint -> 5v TestPoint
- TP4: value 5v TestPoint -> 3v3 TestPoint
- renumbered TP1 to TP5, TP5 to TP6
Connections:
- net 12V_BUS: now also D2.2 (A), J4.5 (Pin_5)
- net 24V_BUS: now also D1.2 (A), J4.1 (Pin_1), TP1.1; no longer TP3.1
- net 3V3_BUS: now also TP4.1, D4.2 (A), J7.4 (VDD)
- net 5V_BUS: now also TP3.1, D3.2 (A), J4.3 (Pin_3); no longer TP4.1
- net BIAS_VOLTAGE: now also J3.2 (Pin_2)
- net CLK: now also U3.5 (A4), J7.5 (CLK); no longer U3.4 (A3)
- net CS: now also U3.1 (A1), J7.2 (DAT3/CD); no longer U3.3 (A2)
- net D_{IN}: now also U3.4 (A3), J7.3 (CMD); no longer U3.1 (A1)
- net GND: now also J3.1 (Pin_1), J7.6 (VSS), J7.9 (SHIELD), R10.1, R11.1, R12.1, R13.1
- net R_SET_A: now also C1.1, R1.2, R4.2
- net R_SET_B: now also C1.2, J3.5 (Pin_5)
- net SENSOR_POWER: now also J4.2 (Pin_2)
- net at R8.2: now also U3.16 (B4); no longer U3.17 (B3)
- net at TP5.1, U1.6 (-), U1.7: now also J3.3 (Pin_3)
- net at R7.2: now also U3.20 (B1); no longer U3.18 (B2)
- net MISO: now reaches XA1.D11
- net MISO: now also R9.1
- net at R5.2: now also U3.17 (B3); no longer U3.20 (B1)
- new net: J3.4 (Pin_4), R4.1
- new net: D4.1 (K), R13.2
- new net: D1.1 (K), R10.2
- new net: J3.6 (Pin_6), R1.1
- new net: D2.1 (K), R11.2
- new net: R9.2, U3.18 (B2)
- new net: D3.1 (K), R12.2
- new net D_{OUT}: J7.7 (DAT0), U3.3 (A2)
- no-connect marks 4 -> 14
Other:
- note added: "SD Card Interface"
- note added: "Transimpediance Amplifier"
- note removed: "Transimpediance Amplifyer"
- moved on the sheet: C3, C4, R5, R6, R7, U3

Commit message: finished PCB design
Parts:
- C1: value 470r -> 470n
Changed lines of the file:
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@@
       (effects (font (size 1.27 1.27)))
     )
-    (property "Value" "470r" (at 229.87 25.4 90)
+    (property "Value" "470n" (at 229.87 25.4 90)
       (effects (font (size 1.27 1.27)))
     )
